File: ArduinoMega2560_RadioController/ArduinoMega2560_RadioController_schema/ArduinoMega2560_RadioController.kicad_sch (KiCad schematic)
At the start: 14 parts

Commit message: modifiche
Parts:
- added A?: MPU6050_Module, Charleslabs_Parts:MPU6050_Module, symbol Charleslabs_Parts:MPU6050_Module
- added C? (x3): 10uF, symbol Device:C
- added C? (x2): 100nF, symbol Device:C
- added D? (x3): 1N4148, Diode_THT:D_DO-35_SOD27_P7.62mm_Horizontal, symbol Diode:1N4148
- added J?: SD_Card, symbol Connector:SD_Card
- added Q? (x2): BC547, Package_TO_SOT_THT:TO-92_Inline, symbol Transistor_BJT:BC547
- added R? (x6): 10k, symbol Device:R
- added R? (x2): 12k, symbol Device:R
- added U?: LM1117-3.3, symbol Regulator_Linear:LM1117-3.3
- R?: value (none) -> 10k
- U?: value (none) -> Joystick5
- U?: value (none) -> Joystick4
- U?: value (none) -> Joystick6
- U?: value (none) -> Joystick2
- U?: value (none) -> NRF24L01_Breakout; footprint (none) -> RF_Module:nRF24L01_Breakout
- U?: value (none) -> Joystick1; footprint (none) -> XDCR_COM-09032
- U?: value (none) -> Joystick3
Connections:
- net +3V3: now also C?.1
- net +5V: now also A?.1 (VCC), C?.1, C?.1, R?.1, U?.3 (VI)
- net GND: now also A?.2 (GND), C?.2, C?.2, C?.2, C?.2, C?.2, J?.12 (SHELL1), J?.13 (SHELL2), J?.3 (VSS), J?.6 (VSS), Q?.3 (E), Q?.3 (E), U?.1 (GND)
- net MISO: now also Q?.1 (C), R?.2
- net MOSI: now also D?.1 (K)
- net NRF_EN: now also A?.D49; no longer A?.D21 (D21/SCL)
- net SCK: now also D?.1 (K)
- net NRF_IRQ: now reaches U?.8 (IRQ)
- net NRF_IRQ: now also A?.D2 (D2_INT0)
- net VbatSens: now reaches A?.A12
- net SDA: now reaches A?.D20 (D20/SDA)
- net SDA: now also A?.4 (SDA)
- net CSN_SD: now reaches A?.D47
- net CSN_SD: now also D?.1 (K)
- new net: C?.1, C?.1, J?.4 (VDD), R?.1, R?.1, R?.1, R?.1, R?.1, R?.2, U?.2 (VO)
- new net: D?.2 (A), J?.1 (CD/DAT3), R?.2
- new net: Q?.2 (B), R?.1
- new net: J?.7 (DAT0), R?.2, R?.2
- new net: D?.2 (A), J?.5 (CLK), R?.2
- new net: Q?.1 (C), Q?.2 (B), R?.1
- new net: D?.2 (A), J?.2 (CMD), R?.2
- new net: J?.8 (DAT1), J?.9 (DAT2), R?.2
- new net SCL: A?.3 (SCL), A?.D21 (D21/SCL)
- no-connect marks 0 -> 12
Other:
- note added: "AD0 => address from 0x68 to 0x69"
- note added: "HEF min:90"
- note added: "Modifiche per SPI a 5v"
- note added: "NRF Module"
- note added: "SCD Card Module"
- moved on the sheet: A?, U?

Commit message: Aggiunto zener e power regulators
Parts:
- removed Q? (x2): BC547, Package_TO_SOT_THT:TO-92_Inline, symbol Transistor_BJT:BC547
- removed R?: 12k, symbol Device:R
- removed R?: 10k, symbol Device:R
- added C1: 470uF, symbol Device:C
- added C2, C4: 100nF, symbol Device:C
- added C3: 100uF, symbol Device:C
- added D1: 3v7/3v3, symbol Device:D_Zener
- added SW1: SW_DPDT_x2, symbol Switch:SW_DPDT_x2
- added U1: L7805, symbol Regulator_Linear:L7805
- added U2: L78L33_TO92, Package_TO_SOT_THT:TO-92_Inline, symbol Regulator_Linear:L78L33_TO92
Connections:
- net +5V: now also C3.1, C4.1, U1.3 (OUT), U2.3 (VI)
- net GND: now also D1.2 (A)
- net MISO: now also R?.1
- net at D?.2 (A), J?.1 (CD/DAT3), R?.2: now also D?.2 (A), D?.2 (A), J?.2 (CMD), J?.5 (CLK), R?.2, R?.2
- net at J?.7 (DAT0), R?.2, R?.2: now also D1.1 (K)
- new net: C1.1, C2.1, SW1.3 (C), U1.1 (IN)
- new net: C1.2, C2.2, C3.2, C4.2, U1.2 (GND), U2.2 (GND)
- new net +12V: SW1.2 (B)
- new net +3.3V: U2.1 (VO)
Other:
- note removed: "HEF min:90"
- moved on the sheet: D?, R?
